Commit message: cleanup and add new launch

File: my_robot/urdf/my_robot.xacro (robot description, xacro)
@@ -188,3 +188,10 @@
     <axis xyz="0 1 0" rpy="0 0 0"/>
   </joint>
+  <joint name="camera_optical_joint" type="fixed">
+    <origin xyz="0 0 0" rpy="-1.5707 0 -1.5707"/>
+    <parent link="camera_link"/>
+    <child link="camera_link_optical"/>
+  </joint>
+  <link name="camera_link_optical">
+  </link>
 </robot>

Commit message: fix camera link

File: my_robot/urdf/my_robot.xacro (robot description, xacro)
@@ -130,5 +130,5 @@
     <dynamics damping="1.0" friction="1.0"/>
   </joint>
-  <link name="camera">
+  <link name="camera_link">
     <inertial>
       <mass value="0.1"/>
@@ -140,5 +140,5 @@
       />
     </inertial>
-    <collision name='camera_collision'>
+    <collision name='camera_link_collision'>
       <origin xyz="0 0 0" rpy=" 0 0 0"/>
       <geometry>
@@ -146,5 +146,5 @@
       </geometry>
     </collision>
-    <visual name='camera_visual'>
+    <visual name='camera_link_visual'>
       <origin xyz="0 0 0" rpy=" 0 0 0"/>
       <geometry>
@@ -155,8 +155,15 @@
   <joint type="fixed" name="camera_joint">
     <origin xyz="0.2 0 0" rpy="0 0 0"/>
-    <child link="camera"/>
+    <child link="camera_link"/>
     <parent link="chassis"/>
     <axis xyz="0 1 0" rpy="0 0 0"/>
   </joint>
+  <joint name="camera_optical_joint" type="fixed">
+    <origin xyz="0 0 0" rpy="-1.5707 0 -1.5707"/>
+    <parent link="camera_link"/>
+    <child link="camera_link_optical"/>
+  </joint>
+  <link name="camera_link_optical">
+  </link>
   <link name="hokuyo">
     <inertial>
@@ -188,10 +195,3 @@
     <axis xyz="0 1 0" rpy="0 0 0"/>
   </joint>
-  <joint name="camera_optical_joint" type="fixed">
-    <origin xyz="0 0 0" rpy="-1.5707 0 -1.5707"/>
-    <parent link="camera_link"/>
-    <child link="camera_link_optical"/>
-  </joint>
-  <link name="camera_link_optical">
-  </link>
 </robot>

Commit message: try to fox

File: my_robot/urdf/my_robot.xacro (robot description, xacro)
@@ -166,4 +166,10 @@
   <link name="camera_link_optical">
   </link>
+  <link name="camera_rgbd_frame"></link>
+  <joint name="camera_rgbd_joint" type="fixed">
+    <origin xyz="0 0 0" rpy="-${pi/2} 0 -${pi/2}"/>
+    <parent link="camera_link"/>
+    <child link="camera_rgbd_frame"/>
+  </joint>
   <link name="hokuyo">
     <inertial>

Commit message: WIP

File: my_robot/urdf/my_robot.xacro (robot description, xacro)
@@ -159,4 +159,6 @@
     <axis xyz="0 1 0" rpy="0 0 0"/>
   </joint>
+  <link name="camera_link_optical">
+  </link>
   <joint name="camera_optical_joint" type="fixed">
     <origin xyz="0 0 0" rpy="-1.5707 0 -1.5707"/>
@@ -164,6 +166,4 @@
     <child link="camera_link_optical"/>
   </joint>
-  <link name="camera_link_optical">
-  </link>
   <link name="camera_rgbd_frame"></link>
   <joint name="camera_rgbd_joint" type="fixed">
